File: CNC.kicad_pcb (KiCad board)
At the start: 2 copper layers, 76.2 x 104.1 mm, 4 parts, among them J1 DRIVER X, J2 DRIVER Y, J3 DRIVER Z

Commit message: Atualização
Parts:
- added REF**: KiCad-Logo2_20mm_Copper, Symbol:KiCad-Logo2_20mm_Copper, F.Cu at (160.0, 135.9)
Other:
- board text removed: "Escola SENAI "LUIZ VARGA Placa CNC GABRIEL MAXIMO DA SILVA"
