File: CNC REVERSA.kicad_pcb (KiCad board)
At the start: 2 copper layers, 76.2 x 104.1 mm, 5 parts, among them J1 DRIVER X, J2 DRIVER Y, J3 DRIVER Z

Commit message: UP
Parts:
- removed REF**: KiCad-Logo2_8mm_B.CU, Symbol:KiCad-Logo2_8mm_B.CU
- moved A1 182.1 mm to (52.1, -35.6)
- moved J1 182.1 mm to (10.2, -38.1)
- moved J2 182.1 mm to (10.2, -6.35)
- moved J3 182.1 mm to (10.2, -71.1)
Routing:
- net GND-Diver: track 0.00 -> 380.1 mm, vias 0 -> 4
- net Dir-Z: track 49.2 -> 65.3 mm
- net Step-Z: track 46.5 -> 62.2 mm
- removed copper zone on B.Cu, net GND-Diver
Other:
- board text added: "ENA X"
- board text added: "ENA Y"
- board text added: "ENA Z"
- board text added: "PUL X"
- board text added: "PUL Y"
- board text added: "PUL Z"
- board text removed: "PLACA CNC ESCOLA SENAI "LUIZ VARGA" GABRIEL MAXIMO DA SILVA"
- board text removed: "STEP Y"
- board text removed: "STEP Z"
- board text removed: "STEPPER X"
- board text removed: "STEPPER Y"
- board text removed: "STEPPER Z"
